Commit message: Feat: added new Kinematic logic + started camera logic

File: robot_urdf/robot_fixed.urdf (robot description, URDF)
Before this commit: robot robot_urdf, 7 links, 6 joints
Joints:
- joint base: limit lower=-3.141592653589793 upper=3.141592653589793 effort=10 velocity=10 -> lower=0 upper=4.27605669661414 effort=10 velocity=10
